File: light_reenginiring.kicad_sch (KiCad schematic)
At the start: 13 parts, among them SW1 SW_SPDT

Commit message: add name of diod bridge
Parts:
- U1: value ~ -> MB10F
Changed lines of the file:
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@@
 			)
 		)
-		(property "Value" "~"
+		(property "Value" "MB10F"
 			(at 54.61 36.83 0)
 			(effects

Commit message: check Voltage
Connections:
- net +V renamed 17.8V
Other:
- note added: "17.8V -> 15V"
- note added: "4.5V"
- note removed: "Idk what voltage on output after converter I think it's 60-80V but need to find proof"
- moved on the sheet: D1, D2, D3, D4, D5, D6, R2
